Commit message: 新增：智元X1接入+机身配色系统+行星减速器动画等十项功能
- 接入智元灵犀X1（52个官方STL+URDF改27可动关节，默认机型）
- 机身配色系统：银白/纯白/金属/原配色/半透明五档可切换，修复金属材质发黑（RoomEnvironment环境贴图）
- 三种减速器原理动画补全行星减速器讲解
- H1/G1同屏对比、拆解顺序动画、力控仿真、拟人步态动画
- 侧边栏拖宽、手机适配、导航无3D标注
- 新增硬件原理图PCB学习页（X1+Hdrive）、参考资料按部位分类

File: 00_解剖式知识可视化/models/x1/x1.urdf (robot description, URDF)
Before this commit: robot x1, 58 links, 57 joints
Joints:
- joint left_elbow_pitch_joint: limit lower=-3.14 upper=3.14 effort=0 velocity=0 -> lower=-1.80 upper=1.80 effort=40 velocity=10; type fixed -> revolute
- joint left_elbow_yaw_joint: limit lower=-3.14 upper=3.14 effort=0 velocity=0 -> lower=-1.00 upper=1.00 effort=40 velocity=10; type fixed -> revolute
- joint left_shoulder_pitch_joint: limit lower=-3.14 upper=3.14 effort=0 velocity=0 -> lower=-2.50 upper=1.80 effort=40 velocity=10; type fixed -> revolute
- joint left_shoulder_roll_joint: limit lower=-3.14 upper=3.14 effort=0 velocity=0 -> lower=-1.20 upper=1.20 effort=40 velocity=10; type fixed -> revolute
- joint left_shoulder_yaw_joint: limit lower=-3.14 upper=3.14 effort=0 velocity=0 -> lower=-1.50 upper=1.50 effort=40 velocity=10; type fixed -> revolute
- joint left_wrist_pitch_joint: limit lower=-3.14 upper=3.14 effort=0 velocity=0 -> lower=-0.90 upper=0.90 effort=40 velocity=10; type fixed -> revolute
- joint lumber_pitch_joint: limit lower=-3.14 upper=3.14 effort=0 velocity=0 -> lower=-0.52 upper=0.52 effort=40 velocity=10; type fixed -> revolute
- joint lumber_roll_joint: limit lower=-3.14 upper=3.14 effort=0 velocity=0 -> lower=-0.52 upper=0.52 effort=40 velocity=10; type fixed -> revolute
- joint lumber_yaw_joint: limit lower=-3.14 upper=3.14 effort=0 velocity=0 -> lower=-0.80 upper=0.80 effort=40 velocity=10; type fixed -> revolute
- joint right_elbow_pitch_joint: limit lower=-3.14 upper=3.14 effort=0 velocity=0 -> lower=-1.80 upper=1.80 effort=40 velocity=10; type fixed -> revolute
- joint right_elbow_yaw_joint: limit lower=-3.14 upper=3.14 effort=0 velocity=0 -> lower=-1.00 upper=1.00 effort=40 velocity=10; type fixed -> revolute
- joint right_shoulder_pitch_joint: limit lower=-3.14 upper=3.14 effort=0 velocity=0 -> lower=-2.50 upper=1.80 effort=40 velocity=10; type fixed -> revolute
- joint right_shoulder_roll_joint: limit lower=-3.14 upper=3.14 effort=0 velocity=0 -> lower=-1.20 upper=1.20 effort=40 velocity=10; type fixed -> revolute
- joint right_shoulder_yaw_joint: limit lower=-3.14 upper=3.14 effort=0 velocity=0 -> lower=-1.50 upper=1.50 effort=40 velocity=10; type fixed -> revolute
- joint right_wrist_pitch_joint: limit lower=-3.14 upper=3.14 effort=0 velocity=0 -> lower=-0.90 upper=0.90 effort=40 velocity=10; type fixed -> revolute
